Commit message: [WIP] Added arbitrary trajectory data collection fields

File: assets/contactnets_cube.urdf (robot description, URDF)
Before this commit: robot cube, 1 links, 0 joints
Links:
- removed link body
- added link cube_body, mass 0.37; collision box size=0.1048 0.1048 0.1048; visual box size=0.1048 0.1048 0.1048

Commit message: [WIP] Set up 2D problem by fixing cube to the XZ plane and the robot fingers to the shifted X axis

File: assets/contactnets_cube.urdf (robot description, URDF)
Before this commit: robot cube, 1 links, 0 joints
Links:
- added link worldfixed
Joints:
- added joint worldfixed_to_cube_body: type planar, parent worldfixed, child cube_body, axis 0 -1 0

Commit message: Working loss landscape plotting Jupyter notebook

File: assets/contactnets_cube.urdf (robot description, URDF)
Before this commit: robot cube, 2 links, 1 joints
Links:
- link cube_body: mass 0.37 -> 0.5; geometry collision box size=0.1 0.1 0.1; visual box size=0.1 0.1 0.1
