Commit message: [WIP] Scaled deviation term by mu, add 'bad' URDF initialization

File: assets/contactnets_cube_bad_init.urdf (robot description, URDF)
Before this commit: robot cube, 1 links, 0 joints
Links:
- removed link body
- added link cube_body, mass 0.37; collision box size=0.1048 0.1048 0.01; visual box size=0.1048 0.1048 0.01
- added link worldfixed
Joints:
- added joint worldfixed_to_cube_body: type planar, parent worldfixed, child cube_body, axis 0 -1 0

Commit message: [WIP] Working on deviation loss function

File: assets/contactnets_cube_bad_init.urdf (robot description, URDF)
Before this commit: robot cube, 2 links, 1 joints
Links:
- link cube_body: geometry collision box size=0.1 0.1 0.1; visual box size=0.1 0.1 0.1
