Commit message: WORKING. Reset weights to previous working state, improve phi calculation to prevent numerical shrinkage artifacts

File: assets/spherebot.urdf (robot description, URDF)
Before this commit: robot spherebot, 7 links, 6 joints
Joints:
- joint finger_0_to_base_z: origin xyz=0 0 0.0524 -> xyz=0 0 0.05
- joint finger_1_to_base_z: origin xyz=0 0 0.0524 -> xyz=0 0 0.05
